Commit message: add lift2s hardware in arx-ros2-control

File: external/arx5-sdk/models/X5.urdf (robot description, URDF)
Before this commit: robot X5, 8 links, 7 joints
Links:
- link base_link: geometry 
- link link1: geometry 
- link link2: geometry 
- link link3: geometry 
- link link4: geometry 
- link link5: geometry 
- link link6: geometry 
