Commit message: Revert "Feature/acone mit：Add MIT MIX arm control and Lift2S lift hardware interface"

File: external/arx5-sdk/models/X5_no_gripper.urdf (robot description, URDF)
Before this commit: robot X5, 8 links, 7 joints
Links:
- link link1: geometry collision mesh filename=./meshes/link1.STL; visual mesh filename=./meshes/link1.STL
- link link2: geometry collision mesh filename=./meshes/link2.STL; visual mesh filename=./meshes/link2.STL
- link link3: geometry collision cylinder length=0.15 radius=0.02; visual mesh filename=./meshes/link3.STL
- link link4: geometry collision cylinder length=0.05 radius=0.025; visual mesh filename=./meshes/link4.STL
- link link5: geometry collision cylinder length=0.025 radius=0.02; visual mesh filename=./meshes/link5.STL
- link link6: mass 0.581000 -> 0.14; geometry collision mesh filename=./meshes/arx_gopro_finray_gripper.stl; visual mesh filename=./meshes/arx_gopro_finray_gripper.stl
Joints:
- joint gripper_fixed_joint: origin xyz=0.145 0.0 0.0 rpy=0 0 0 -> xyz=0.185 0.0 0.0 rpy=0 0 0
- joint joint6: limit lower=-1.57 upper=1.57 effort=100 velocity=1000 -> lower=-1.57 upper=1.57 effort=30 velocity=10

File: external/arx5-sdk/models/X5_umi.urdf (robot description, URDF)
Before this commit: robot X5, 8 links, 7 joints
Links:
- link base_link: geometry collision mesh filename=./meshes/X5/base_link.STL; visual mesh filename=./meshes/X5/base_link.STL
- link eef_link: mass 0.0 -> 0.0001
- link link6: mass 0.581000 -> 0.902; geometry collision mesh filename=./meshes/arx_gopro_finray_gripper.stl; visual mesh filename=./meshes/arx_gopro_finray_gripper.stl
Joints:
- joint gripper_fixed_joint: origin xyz=0.145 0.0 0.0 rpy=0 0 0 -> xyz=0.225 0.0 0.0 rpy=0 0 0
- joint joint6: limit lower=-1.57 upper=1.57 effort=100 velocity=1000 -> lower=-1.57 upper=1.57 effort=30 velocity=10
